File: ESPProgrammer.sch (EAGLE design)
At the start: 3 parts

Commit message: update file
Parts:
- added JP3: (no value), pinhead:PINHD-1X4
- added JP4, JP5: (no value), pinhead:PINHD-1X8
- added JP6: (no value), pinhead:PINHD-1X2
Connections:
- new net N$1: JP3.1, JP5.5, U1.GPIO0
- new net N$10: JP4.7, U1.ADC
- new net N$11: JP4.5, U1.GPIO16
- new net N$12: JP4.4, U1.GPIO14
- new net N$13: JP4.3, U1.GPIO12
- new net N$14: JP4.2, U1.GPIO13
- new net N$15: JP4.6, JP6.1, U1.CH_PD
- new net N$2: JP3.4, JP5.7, U1.GPIO15
- new net N$3: JP5.3, U1.GPIO4
- new net N$6: JP5.4, U1.GPIO5
- new net N$7: JP5.6, U1.GPIO2
- new net N$9: JP4.8, U1.RESET
- net GND: now also JP3.2, JP3.3, JP5.8; no longer U1.GPIO0, U1.GPIO15
- net N$4: now also JP5.2
- net N$5: now also JP5.1
- net VCC: now also JP4.1, JP6.2; no longer U1.CH_PD
Changed lines of the file:
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@@
 <setting verticaltext="up"/>
 </settings>
-<grid distance="0.1" unitdist="inch" unit="inch" style="lines" multiple="1" display="no" altdistance="0.01" altunitdist="inch" altunit="inch"/>
+<grid distance="0.1" unitdist="inch" unit="mm" style="lines" multiple="1" display="no" altdistance="0.01" altunitdist="inch" altunit="mm"/>
 <layers>
 <layer number="1" name="Top" color="4" fill="1" visible="no" active="no"/>
@@
 </variantdefs>
 <classes>
-<class number="0" name="default" width="0.5" drill="0.6">
-<clearance class="0" value="0.5"/>
+<class number="0" name="default" width="0.7" drill="0.6">
+<clearance class="0" value="0.4"/>
 </class>
 </classes>
@@
 <part name="P+3" library="supply1" deviceset="VCC" device=""/>
 <part name="U1" library="esp8266modules" deviceset="ESP12" device=""/>
+<part name="JP3" library="pinhead" deviceset="PINHD-1X4" device=""/>
+<part name="JP4" library="pinhead" deviceset="PINHD-1X8" device=""/>
+<part name="JP5" library="pinhead" deviceset="PINHD-1X8" device=""/>
+<part name="JP6" library="pinhead" deviceset="PINHD-1X2" device=""/>
 </parts>
 <sheets>
@@
 <instance part="P+3" gate="VCC" x="43.18" y="5.08"/>
 <instance part="U1" gate="G$1" x="66.04" y="12.7"/>
+<instance part="JP3" gate="A" x="73.66" y="-38.1" rot="R270"/>
+<instance part="JP4" gate="A" x="27.94" y="12.7" rot="R180"/>
+<instance part="JP5" gate="A" x="114.3" y="10.16"/>
+<instance part="JP6" gate="G$1" x="45.72" y="-38.1" rot="R270"/>
 </instances>
 <busses>
@@
 <wire x1="86.36" y1="17.78" x2="81.28" y2="17.78" width="0.1524" layer="91"/>
 <pinref part="U1" gate="G$1" pin="RX"/>
+<pinref part="JP5" gate="A" pin="2"/>
+<wire x1="86.36" y1="17.78" x2="111.76" y2="17.78" width="0.1524" layer="91"/>
 </segment>
 </net>
@@
 <wire x1="81.28" y1="25.4" x2="81.28" y2="20.32" width="0.1524" layer="91"/>
 <pinref part="U1" gate="G$1" pin="TX"/>
+<pinref part="JP5" gate="A" pin="1"/>
+<wire x1="81.28" y1="20.32" x2="111.76" y2="20.32" width="0.1524" layer="91"/>
 </segment>
 </net>
@@
 </segment>
 <segment>
-<wire x1="81.28" y1="10.16" x2="86.36" y2="10.16" width="0.1524" layer="91"/>
-<wire x1="86.36" y1="10.16" x2="86.36" y2="5.08" width="0.1524" layer="91"/>
-<wire x1="81.28" y1="5.08" x2="86.36" y2="5.08" width="0.1524" layer="91"/>
 <pinref part="GND3" gate="1" pin="GND"/>
 <wire x1="86.36" y1="5.08" x2="93.98" y2="5.08" width="0.1524" layer="91"/>
@@
 <wire x1="86.36" y1="2.54" x2="81.28" y2="2.54" width="0.1524" layer="91"/>
 <pinref part="U1" gate="G$1" pin="GND"/>
-<pinref part="U1" gate="G$1" pin="GPIO15"/>
-<pinref part="U1" gate="G$1" pin="GPIO0"/>
+<wire x1="93.98" y1="5.08" x2="101.6" y2="5.08" width="0.1524" layer="91"/>
+<wire x1="101.6" y1="5.08" x2="101.6" y2="-7.62" width="0.1524" layer="91"/>
+<pinref part="JP3" gate="A" pin="2"/>
+<wire x1="101.6" y1="-7.62" x2="76.2" y2="-7.62" width="0.1524" layer="91"/>
+<wire x1="76.2" y1="-7.62" x2="76.2" y2="-35.56" width="0.1524" layer="91"/>
+<pinref part="JP3" gate="A" pin="3"/>
+<wire x1="76.2" y1="-35.56" x2="73.66" y2="-35.56" width="0.1524" layer="91"/>
+<wire x1="101.6" y1="5.08" x2="104.14" y2="5.08" width="0.1524" layer="91"/>
+<wire x1="104.14" y1="5.08" x2="104.14" y2="2.54" width="0.1524" layer="91"/>
+<pinref part="JP5" gate="A" pin="8"/>
+<wire x1="104.14" y1="2.54" x2="111.76" y2="2.54" width="0.1524" layer="91"/>
 </segment>
 </net>
@@
 </segment>
 <segment>
+<pinref part="JP4" gate="A" pin="1"/>
+<pinref part="P+3" gate="VCC" pin="VCC"/>
+<pinref part="U1" gate="G$1" pin="VCC"/>
 <wire x1="48.26" y1="2.54" x2="45.72" y2="2.54" width="0.1524" layer="91"/>
-<pinref part="P+3" gate="VCC" pin="VCC"/>
-<wire x1="45.72" y1="2.54" x2="43.18" y2="2.54" width="0.1524" layer="91"/>
-<wire x1="48.26" y1="15.24" x2="45.72" y2="15.24" width="0.1524" layer="91"/>
-<wire x1="45.72" y1="15.24" x2="45.72" y2="2.54" width="0.1524" layer="91"/>
+<wire x1="43.18" y1="2.54" x2="30.48" y2="2.54" width="0.1524" layer="91"/>
+<pinref part="JP6" gate="G$1" pin="2"/>
+<wire x1="43.18" y1="2.54" x2="45.72" y2="2.54" width="0.1524" layer="91"/>
+<wire x1="45.72" y1="2.54" x2="45.72" y2="-35.56" width="0.1524" layer="91"/>
+</segment>
+</net>
+<net name="N$1" class="0">
+<segment>
+<pinref part="U1" gate="G$1" pin="GPIO0"/>
+<pinref part="JP3" gate="A" pin="1"/>
+<wire x1="81.28" y1="10.16" x2="78.74" y2="10.16" width="0.1524" layer="91"/>
+<wire x1="78.74" y1="10.16" x2="78.74" y2="-35.56" width="0.1524" layer="91"/>
+<pinref part="JP5" gate="A" pin="5"/>
+<wire x1="111.76" y1="10.16" x2="81.28" y2="10.16" width="0.1524" layer="91"/>
+</segment>
+</net>
+<net name="N$2" class="0">
+<segment>
+<pinref part="U1" gate="G$1" pin="GPIO15"/>
+<wire x1="81.28" y1="5.08" x2="81.28" y2="-5.08" width="0.1524" layer="91"/>
+<pinref part="JP3" gate="A" pin="4"/>
+<wire x1="81.28" y1="-5.08" x2="71.12" y2="-5.08" width="0.1524" layer="91"/>
+<wire x1="71.12" y1="-5.08" x2="71.12" y2="-35.56" width="0.1524" layer="91"/>
+<pinref part="JP5" gate="A" pin="7"/>
+<wire x1="111.76" y1="5.08" x2="109.22" y2="5.08" width="0.1524" layer="91"/>
+<wire x1="111.76" y1="5.08" x2="119.38" y2="5.08" width="0.1524" layer="91"/>
+<wire x1="119.38" y1="5.08" x2="119.38" y2="-20.32" width="0.1524" layer="91"/>
+<wire x1="119.38" y1="-20.32" x2="71.12" y2="-20.32" width="0.1524" layer="91"/>
+<wire x1="71.12" y1="-20.32" x2="71.12" y2="-35.56" width="0.1524" layer="91"/>
+</segment>
+</net>
+<net name="N$3" class="0">
+<segment>
+<pinref part="U1" gate="G$1" pin="GPIO4"/>
+<pinref part="JP5" gate="A" pin="3"/>
+<wire x1="81.28" y1="15.24" x2="111.76" y2="15.24" width="0.1524" layer="91"/>
+</segment>
+</net>
+<net name="N$6" class="0">
+<segment>
+<pinref part="U1" gate="G$1" pin="GPIO5"/>
+<pinref part="JP5" gate="A" pin="4"/>
+<wire x1="81.28" y1="12.7" x2="111.76" y2="12.7" width="0.1524" layer="91"/>
+</segment>
+</net>
+<net name="N$7" class="0">
+<segment>
+<pinref part="JP5" gate="A" pin="6"/>
+<pinref part="U1" gate="G$1" pin="GPIO2"/>
+<wire x1="111.76" y1="7.62" x2="81.28" y2="7.62" width="0.1524" layer="91"/>
+</segment>
+</net>
+<net name="N$9" class="0">
+<segment>
+<pinref part="U1" gate="G$1" pin="RESET"/>
+<pinref part="JP4" gate="A" pin="8"/>
+<wire x1="48.26" y1="20.32" x2="30.48" y2="20.32" width="0.1524" layer="91"/>
+</segment>
+</net>
+<net name="N$10" class="0">
+<segment>
+<pinref part="U1" gate="G$1" pin="ADC"/>
+<pinref part="JP4" gate="A" pin="7"/>
+<wire x1="48.26" y1="17.78" x2="30.48" y2="17.78" width="0.1524" layer="91"/>
+</segment>
+</net>
+<net name="N$11" class="0">
+<segment>
+<pinref part="U1" gate="G$1" pin="GPIO16"/>
+<pinref part="JP4" gate="A" pin="5"/>
+<wire x1="48.26" y1="12.7" x2="30.48" y2="12.7" width="0.1524" layer="91"/>
+</segment>
+</net>
+<net name="N$12" class="0">
+<segment>
+<pinref part="U1" gate="G$1" pin="GPIO14"/>
+<pinref part="JP4" gate="A" pin="4"/>
+<wire x1="48.26" y1="10.16" x2="30.48" y2="10.16" width="0.1524" layer="91"/>
+</segment>
+</net>
+<net name="N$13" class="0">
+<segment>
+<pinref part="U1" gate="G$1" pin="GPIO12"/>
+<pinref part="JP4" gate="A" pin="3"/>
+<wire x1="48.26" y1="7.62" x2="30.48" y2="7.62" width="0.1524" layer="91"/>
+</segment>
+</net>
+<net name="N$14" class="0">
+<segment>
+<pinref part="U1" gate="G$1" pin="GPIO13"/>
+<pinref part="JP4" gate="A" pin="2"/>
+<wire x1="48.26" y1="5.08" x2="30.48" y2="5.08" width="0.1524" layer="91"/>
+</segment>
+</net>
+<net name="N$15" class="0">
+<segment>
 <pinref part="U1" gate="G$1" pin="CH_PD"/>
-<pinref part="U1" gate="G$1" pin="VCC"/>
-</segment>
-</net>
+<pinref part="JP4" gate="A" pin="6"/>
+<wire x1="48.26" y1="15.24" x2="30.48" y2="15.24" width="0.1524" layer="91"/>
+<wire x1="30.48" y1="15.24" x2="20.32" y2="15.24" width="0.1524" layer="91"/>
+<wire x1="20.32" y1="15.24" x2="20.32" y2="-22.86" width="0.1524" layer="91"/>
+<pinref part="JP6" gate="G$1" pin="1"/>
+<wire x1="20.32" y1="-22.86" x2="48.26" y2="-22.86" width="0.1524" layer="91"/>
+<wire x1="48.26" y1="-22.86" x2="48.26" y2="-35.56" width="0.1524" layer="91"/>
+</segment>
+</net>
